File: pi-zero-interconnect/pi-zero-interconnect.kicad_pcb (KiCad board)
At the start: 2 copper layers, 87 x 17 mm, 5 parts, among them J1 Raspberry_Pi_2x20_PTH_NoSilk, J2 PI ZERO

Commit message: REV 0.1.0 intial Release
Parts:
- moved TP1 1.64 mm to (96.2, 107.4)
Routing:
- net Net-(J1-3V3-Pad1): track 26.0 -> 24.3 mm
Other:
- board text added: "PI-ZERO-INTERCONNECT PCBA"
- board text added: "REV: ${REV}"
