File: pi-zero-interconnect/pi-zero-interconnect.kicad_sch (KiCad schematic)
At the start: 5 parts, among them J1 Raspberry_Pi_2x20_PTH_NoSilk, J2 PI ZERO

Commit message: REV 0.1.0 intial Release
Other:
- company: (none) -> Montis Corporation
- title: (none) -> Pi Zero Interconnect
Changed lines of the file:
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@@
 	(generator_version "10.0")
 	(paper "A4")
+	(title_block
+		(title "Pi Zero Interconnect")
+		(date "2026-04-24")
+		(rev "${REV}")
+		(company "Montis Corporation")
+		(comment 1 "Author: Matt White")
+		(comment 2 "Reviewer: --")
+	)
 	(junction
 		(at 168.91 95.25)
